Commit message: feat: update urdf to new calib version

File: urdf/SO101_follower.urdf (robot description, URDF)
Before this commit: robot SO101_follower, 7 links, 6 joints
Links:
- removed link base
- removed link gripper
- removed link jaw
- removed link lower_arm
- removed link shoulder
- removed link upper_arm
- removed link wrist
- added link base_link, mass 0.147; collision mesh filename=package://so101_description/meshes/base_motor_holder_so101_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; collision mesh filename=package://so101_description/meshes/base_so101_v2.stl
- added link gripper_frame_link, mass 1e-9
- added link gripper_link, mass 0.087; collision mesh filename=package://so101_description/meshes/sts3215_03a_v1.stl; collision mesh filename=package://so101_description/meshes/wrist_roll_follower_so10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
- added link lower_arm_link, mass 0.104; collision mesh filename=package://so101_description/meshes/motor_holder_so101_wrist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; collision mesh filename=package://so101_description/meshes/sts3215_03a_v1.stl
- added link moving_jaw_link, mass 0.012; collision mesh filename=package://so101_description/meshes/moving_jaw_so101_v1.stl; visual mesh filename=package://so101_description/meshes/moving_jaw_so101_v1.stl
- added link shoulder_link, mass 0.100006; collision mesh filename=package://so101_description/meshes/motor_holder_so101_base_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; collision mesh filename=package://so101_description/meshes/rotation_pitch_so101_v1.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
- added link upper_arm_link, mass 0.103; collision mesh filename=package://so101_description/meshes/sts3215_03a_v1.stl; collision mesh filename=package://so101_description/meshes/upper_arm_so101_v1.stl
- added link wrist_link, mass 0.079; collision mesh filename=package://so101_description/meshes/sts3215_03a_no_horn_v1.s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; collision mesh filename=package://so101_description/meshes/wrist_roll_pitch_so101_v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
Joints:
- added joint gripper_frame_joint: type fixed, parent gripper_link, child gripper_frame_link, origin xyz=-0.0079 -0.000218121 -0.0981274 rpy=0 3.14159 0, axis 0 0 0
- joint elbow_flex: child lower_arm -> lower_arm_link; limit lower=-0.174533 upper=3.14159 effort=10 velocity=10 -> lower=-1.69 upper=1.69 effort=10 velocity=10; origin xyz=-0.028 0.11257 1.24466e-16 rpy=1.89432e-15 -3.22659e-15 -3.14159 -> xyz=-0.11257 -0.028 1.73763e-16 rpy=-3.63608e-16 8.74301e-16 1.5708; parent upper_arm -> upper_arm_link
- joint gripper: child jaw -> moving_jaw_link; origin xyz=0.0202 0.0188 -0.0234 rpy=1.5708 -7.91661e-17 -1.0396e-16 -> xyz=0.0202 0.0188 -0.0234 rpy=1.5708 -5.24284e-08 -1.41553e-15; parent gripper -> gripper_link
- joint shoulder_lift: child upper_arm -> upper_arm_link; limit lower=-3.31613 upper=0.174533 effort=10 velocity=10 -> lower=-1.74533 upper=1.74533 effort=10 velocity=10; origin xyz=-0.0303992 -0.0182778 -0.0542 rpy=-1.5708 1.5708 0 -> xyz=-0.0303992 -0.0182778 -0.0542 rpy=-1.5708 -1.5708 0; parent shoulder -> shoulder_link
- joint shoulder_pan: child shoulder -> shoulder_link; origin xyz=0.0207909 -0.0230745 0.0948817 rpy=-3.14159 6.03684e-16 1.5708 -> xyz=0.0388353 -8.97657e-09 0.0624 rpy=3.14159 4.18253e-17 -3.14159; parent base -> base_link
- joint wrist_flex: child wrist -> wrist_link; origin xyz=-0.0052 -0.1349 3.40439e-16 rpy=-1.41553e-15 4.91611e-15 7.56157e-09 -> xyz=-0.1349 0.0052 3.62355e-17 rpy=4.02456e-15 8.67362e-16 -1.5708; parent lower_arm -> lower_arm_link
- joint wrist_roll: child gripper -> gripper_link; limit lower=-2.79253 upper=2.79253 effort=10 velocity=10 -> lower=-2.74385 upper=2.84121 effort=10 velocity=10; origin xyz=2.77556e-17 -0.0611 0.0181 rpy=1.5708 -9.38083e-08 3.14159 -> xyz=5.55112e-17 -0.0611 0.0181 rpy=1.5708 0.0486795 3.14159; parent wrist -> wrist_link
